File: dactyl_circuit_right_hand_from_below.sch (KiCad schematic (older format))
At the start: 154 parts, among them SW11 SW_Push, SW12 SW_Push, SW13 SW_Push, SW14 SW_Push, SW15 SW_Push, SW16 SW_Push, SW21 SW_Push, SW22 SW_Push, SW23 SW_Push, SW24 SW_Push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

Commit message: Wiring : redo the matrix properly to follow qmk_firmware. Diode placement within switch to be checked
Parts:
- renumbered D16 to D11, D15 to D12, D14 to D13, D13 to D14, D12 to D15, D11 to D16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
